Commit message: Update depthcam.xacro

File: camera/realsense_ros_gazebo/xacro/depthcam.xacro (robot description, xacro)
@@ -40,9 +40,9 @@
         </geometry>
       </collision>
-      <inertial>
-        <mass value="${d435_cam_mass}" />
-        <origin xyz="0 ${-d435_cam_depth_py} 0" rpy="0 0 0"/>
-        <xacro:box_inertia m="${d435_cam_mass}" x="${d435_cam_depth}" y="${d435_cam_width}" z="${d435_cam_height}"/>
-      </inertial>
+      #<inertial>
+        #<mass value="${d435_cam_mass}" />
+        #<origin xyz="0 ${-d435_cam_depth_py} 0" rpy="0 0 0"/>
+       #<xacro:box_inertia m="${d435_cam_mass}" x="${d435_cam_depth}" y="${d435_cam_width}" z="${d435_cam_height}"/>
+      #</inertial>
     </link>
     <!-- camera depth joints and links -->

Commit message: Update depthcam.xacro

File: camera/realsense_ros_gazebo/xacro/depthcam.xacro (robot description, xacro)
@@ -40,9 +40,9 @@
         </geometry>
       </collision>
-      #<inertial>
-        #<mass value="${d435_cam_mass}" />
-        #<origin xyz="0 ${-d435_cam_depth_py} 0" rpy="0 0 0"/>
-       #<xacro:box_inertia m="${d435_cam_mass}" x="${d435_cam_depth}" y="${d435_cam_width}" z="${d435_cam_height}"/>
-      #</inertial>
+      <!--<inertial>
+        <mass value="${d435_cam_mass}" />
+        <origin xyz="0 ${-d435_cam_depth_py} 0" rpy="0 0 0"/>
+       <xacro:box_inertia m="${d435_cam_mass}" x="${d435_cam_depth}" y="${d435_cam_width}" z="${d435_cam_height}"/>
+      </inertial>-->
     </link>
     <!-- camera depth joints and links -->

Commit message: Update depthcam.xacro

File: camera/realsense_ros_gazebo/xacro/depthcam.xacro (robot description, xacro)
@@ -31,5 +31,5 @@
         <origin xyz="${d435_cam_mount_from_center_offset} ${-d435_cam_depth_py} 0" rpy="${pi/2} 0 ${pi/2}"/>
         <geometry>
-          <mesh filename="/home/iastaff/catkin_ws/src/drone/camera/realsense_ros_gazebo/meshes/realsense_d435.stl" />
+          <mesh filename="package://drone/urdf/meshes/realsense_d435.stl" />
         </geometry>
       </visual>
