Commit message: Update quadrotor_base_with_realsense.urdf.xacro

File: urdf/xacro/quadrotor_base_with_realsense.urdf.xacro (robot description, xacro)
@@ -32,5 +32,5 @@
     <!-- D435I sensor -->
     <xacro:realsense_d435 sensor_name="d435" parent_link="base_link" rate="10" >
-      <origin rpy="0 1.57079632679 0 " xyz="0 0 0.0002"/>
+      <origin rpy="0 0 1.57079632679 " xyz="0 0.1 -0.15"/>
     </xacro:realsense_d435>
   </xacro:macro>

Commit message: Update quadrotor_base_with_realsense.urdf.xacro

File: urdf/xacro/quadrotor_base_with_realsense.urdf.xacro (robot description, xacro)
@@ -32,5 +32,5 @@
     <!-- D435I sensor -->
     <xacro:realsense_d435 sensor_name="d435" parent_link="base_link" rate="10" >
-      <origin rpy="0 0 1.57079632679 " xyz="0 0.1 -0.15"/>
+      <origin rpy="0 0 1.57079632679 " xyz="0 0.1 -0.19"/>
     </xacro:realsense_d435>
   </xacro:macro>
